Commit message: many changes

File: Hands-On_1/robot_arm.urdf (robot description, URDF)
Before this commit: robot table_with_post, 2 links, 1 joints
Links:
- removed link post
- removed link table
- added link cam_bar_link, mass 5.0; collision box size=0.4 0.04 0.04; visual box size=0.4 0.04 0.04
- added link cam_link, mass 5.0; collision box size=0.04 0.08 0.04; visual mesh filename=meshes/d435.dae
- added link cam_post_link, mass 5.0; collision cylinder length=1.0 radius=0.1; visual box size=0.04 0.04 1.0
- added link table_link, mass 10.0; collision box size=1.0 1.5 1.0; visual box size=1.0 1.5 1.0
- added link world
Joints:
- removed joint table_to_post
- added joint cam_post_to_cam_bar_joint: type fixed, parent cam_post_link, child cam_bar_link, origin xyz=0.0 0 0.93
- added joint cam_to_cam_bar_joint: type fixed, parent cam_bar_link, child cam_link, origin xyz=0.2 0 0.0
- added joint table_joint: type fixed, parent world, child table_link, origin xyz=2.0 2.0 0.0
- added joint table_to_cam_post_joint: type fixed, parent table_link, child cam_post_link, origin xyz=-0.4 0 1.0
